File: Collins-FMS-3000.kicad_pcb (KiCad board)
At the start: 2 copper layers, 145 x 161 mm, 131 parts, among them J1 USB_B_Mini, J2 AVR-ISP-6, J3 Conn_02x04_Odd_Even, SW1 SW_Push_LED, SW10 SW_Push_LED, SW11 SW_Push_LED, SW12 SW_Push_LED, SW13 SW_Push_LED, SW14 SW_Push_LED, SW15 SW_Push_LED, SW16 SW_Push_LED, SW17 SW_Push_LED, SW18 SW_Push_LED, SW19 SW_Push_LED, SW2 SW_Push_LED, SW20 SW_Push_LED, SW21 SW_Push_LED, SW22 SW_Push_LED, SW23 SW_Push_LED, SW24 SW_Push_LED, SW25 SW_Push_LED, SW26 SW_Push_LED, SW27 SW_Push_LED, SW28 SW_Push_LED, SW29 SW_Push_LED, SW3 SW_Push_LED, SW30 SW_Push_LED, SW31 SW_Push_LED, SW32 SW_Push_LED, SW33 SW_Push_LED, SW34 SW_Push_LED, SW35 SW_Push_LED, SW36 SW_Push_LED, SW37 SW_Push_LED, SW38 SW_Push_LED, SW39 SW_Push_LED, SW4 SW_Push_LED, SW40 SW_Push_LED, SW41 SW_Push_LED, SW42 SW_Push_LED, SW43 SW_Push_LED, SW44 SW_Push_LED, SW45 SW_Push_LED, SW46 SW_Push_LED, SW47 SW_Push_LED, SW48 SW_Push_LED, SW49 SW_Push_LED, SW5 SW_Push_LED, SW50 SW_Push_LED, SW51 SW_Push_LED, SW52 SW_Push_LED, SW53 SW_Push_LED, SW54 SW_Push_LED, SW55 SW_Push_LED, SW56 SW_Push_LED, SW57 SW_Push_LED, SW58 SW_Push_LED, SW59 SW_Push_LED, SW6 SW_Push_LED, SW60 SW_Push_LED, SW61 SW_Push_LED, SW62 SW_Push_LED, SW63 SW_Push_LED, SW64 SW_Push_LED, SW65 SW_Push_LED, SW66 SW_Push_LED, SW67 SW_Push_LED, SW68 SW_Push_LED, SW69 SW_Push_LED, SW7 SW_Push_LED, SW70 SW_Push, SW8 SW_Push_LED, SW9 SW_Push_LED, U1 ATmega32U4-MU, U2 MCP23017_SO, U3 MCP23017_SO, U4 IS31FL3733B, Y1 16MHz

Commit message: All buttons moved to new layout
Parts:
- removed H14, H15: MountingHole, MountingHole:MountingHole_3.2mm_M3
- removed R26: 330, Collins-FMS-3000:Perfect_0402
- removed SW70: SW_Push, Button_Switch_THT:SW_PUSH_6mm_H4.3mm
- added H5: MountingHole, Collins-FMS-3000:JLCPCB_Tooling_Hole, F.Cu at (25.1, 18.8)
- added H6: MountingHole, Collins-FMS-3000:JLCPCB_Tooling_Hole, F.Cu at (152.6, 19.1)
- added H7: MountingHole, Collins-FMS-3000:JLCPCB_Tooling_Hole, F.Cu at (25.1, 173.0)
- added R10: 2k2, Collins-FMS-3000:Perfect_0402, F.Cu at (170.0, 41.9)
- added R11: 2k2, Collins-FMS-3000:Perfect_0402, F.Cu at (166.9, 46.0)
- added R12: 2k2, Collins-FMS-3000:Perfect_0402, F.Cu at (170.0, 44.0)
- added R13: 2k2, Collins-FMS-3000:Perfect_0402, F.Cu at (173.2, 41.9)
- added R14: 2k2, Collins-FMS-3000:Perfect_0402, F.Cu at (170.0, 46.0)
- added R15: 2k2, Collins-FMS-3000:Perfect_0402, F.Cu at (173.2, 44.0)
- added R16: 2k2, Collins-FMS-3000:Perfect_0402, F.Cu at (176.3, 41.9)
- added R17: 2k2, Collins-FMS-3000:Perfect_0402, F.Cu at (173.2, 46.0)
- added R18: 2k2, Collins-FMS-3000:Perfect_0402, F.Cu at (176.3, 44.0)
- added R19: 2k2, Collins-FMS-3000:Perfect_0402, F.Cu at (176.3, 46.0)
- added R8: 2k2, Collins-FMS-3000:Perfect_0402, F.Cu at (166.9, 41.9)
- added R9: 2k2, Collins-FMS-3000:Perfect_0402, F.Cu at (166.9, 44.0)
- J2: footprint Connector_PinHeader_2.54mm:PinHeader_2x03_P2.54mm_Vertical -> Connector:Tag-Connect_TC2030-IDC-NL_2x03_P1.27mm_Vertical
- moved H12 376.2 mm to (127.0, 76.2)
- moved H1 372.3 mm to (19.6, 172.9)
- moved H11 372.3 mm to (19.5, 97.0)
- moved SW15 372.3 mm to (33.3, 115.7)
- moved SW25 372.3 mm to (63.1, 115.7)
- moved SW36 372.3 mm to (91.9, 128.0)
- moved SW37 372.3 mm to (91.9, 141.5)
- moved SW38 372.3 mm to (91.9, 154.9)
- moved SW39 372.3 mm to (91.9, 168.4)
- moved SW40 372.3 mm to (107.6, 115.7)
- moved SW41 372.3 mm to (104.1, 128.0)
- moved SW42 372.3 mm to (104.1, 141.5)
- moved SW43 372.3 mm to (104.1, 154.9)
- moved SW44 372.3 mm to (104.1, 168.4)
- moved SW46 372.3 mm to (116.3, 128.0)
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Routing:
- net +5V: track 443.2 -> 290.8 mm
- net I2C_SDA: track 276.2 -> 132.2 mm, vias 5 -> 4
- net I2C_SCL: track 281.7 -> 138.5 mm, vias 5 -> 4
- net /LEDMatrix/CS2: track 138.1 -> 8.15 mm, vias 2 -> 1
- net /LEDMatrix/CS5: track 43.6 -> 13.9 mm, vias 2 -> 1
- net /LEDMatrix/CS6: track 43.7 -> 15.1 mm, vias 2 -> 1
- net /LEDMatrix/CS1: track 28.6 -> 8.88 mm, vias 2 -> 1
- net /LEDMatrix/CS4: track 23.2 -> 7.69 mm
- net Net-(R26-Pad2): track 9.45 -> 0.00 mm
- net GND: track 118.7 -> 113.9 mm, vias 35 -> 36
- net /ATmega32u4/SCK: track 11.3 -> 7.49 mm
- net /ButtonMatrix/ROW0: track 27.9 -> 25.7 mm
- net /ButtonMatrix/ROW1: track 34.3 -> 32.1 mm
- net RESET: track 29.2 -> 31.0 mm, vias 0 -> 2
- net /LEDMatrix/SW6: track 55.2 -> 53.8 mm
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Other:
- board text removed: "MISO"
- board text removed: "MOSI"
- board text removed: "RESET"
- board text removed: "SCK"
