File: ButtonMatrix.sch (KiCad schematic (older format))
At the start: 81 parts, among them SW1 SW_Push_LED, SW10 SW_Push_LED, SW11 SW_Push_LED, SW12 SW_Push_LED, SW13 SW_Push_LED, SW14 SW_Push_LED, SW15 SW_Push_LED, SW16 SW_Push_LED, SW17 SW_Push_LED, SW18 SW_Push_LED, SW19 SW_Push_LED, SW2 SW_Push_LED, SW20 SW_Push_LED, SW21 SW_Push_LED, SW22 SW_Push_LED, SW23 SW_Push_LED, SW24 SW_Push_LED, SW25 SW_Push_LED, SW26 SW_Push_LED, SW27 SW_Push_LED, SW28 SW_Push_LED, SW29 SW_Push_LED, SW3 SW_Push_LED, SW30 SW_Push_LED, SW31 SW_Push_LED, SW32 SW_Push_LED, SW33 SW_Push_LED, SW34 SW_Push_LED, SW35 SW_Push_LED, SW36 SW_Push_LED, SW37 SW_Push_LED, SW38 SW_Push_LED, SW39 SW_Push_LED, SW4 SW_Push_LED, SW40 SW_Push_LED, SW41 SW_Push_LED, SW42 SW_Push_LED, SW43 SW_Push_LED, SW44 SW_Push_LED, SW45 SW_Push_LED, SW46 SW_Push_LED, SW47 SW_Push_LED, SW48 SW_Push_LED, SW49 SW_Push_LED, SW5 SW_Push_LED, SW50 SW_Push_LED, SW51 SW_Push_LED, SW52 SW_Push_LED, SW53 SW_Push_LED, SW54 SW_Push_LED, SW55 SW_Push_LED, SW56 SW_Push_LED, SW57 SW_Push_LED, SW58 SW_Push_LED, SW59 SW_Push_LED, SW6 SW_Push_LED, SW60 SW_Push_LED, SW61 SW_Push_LED, SW62 SW_Push_LED, SW63 SW_Push_LED, SW64 SW_Push_LED, SW65 SW_Push_LED, SW66 SW_Push_LED, SW67 SW_Push_LED, SW68 SW_Push_LED, SW69 SW_Push_LED, SW7 SW_Push_LED, SW8 SW_Push_LED, SW9 SW_Push_LED

Commit message: Update components to match JLCPCB availability
Parts:
- R10, R11, R12, R13, R14, R15, R16, R17, R18, R19, R8, R9: footprint Collins-FMS-3000:Perfect_0402 -> Resistor_SMD:R_0603_1608Metric; JLC (none) -> 0603; LCSC (none) -> C22939
Changed lines of the file:
@@
 F 0 "R8" H 3559 1646 50  0000 L CNN
 F 1 "2k2" H 3559 1555 50  0000 L CNN
-F 2 "Collins-FMS-3000:Perfect_0402" H 3500 1600 50  0001 C CNN
+F 2 "Resistor_SMD:R_0603_1608Metric" H 3500 1600 50  0001 C CNN
 F 3 "~" H 3500 1600 50  0001 C CNN
+F 4 "0603" H 3500 1600 50  0001 C CNN "JLC"
+F 5 "C22939" H 3500 1600 50  0001 C CNN "LCSC"
 	1    3500 1600
 	1    0    0    -1
@@
 F 0 "R9" H 3559 1946 50  0000 L CNN
 F 1 "2k2" H 3559 1855 50  0000 L CNN
-F 2 "Collins-FMS-3000:Perfect_0402" H 3500 1900 50  0001 C CNN
+F 2 "Resistor_SMD:R_0603_1608Metric" H 3500 1900 50  0001 C CNN
 F 3 "~" H 3500 1900 50  0001 C CNN
+F 4 "0603" H 3500 1900 50  0001 C CNN "JLC"
+F 5 "C22939" H 3500 1900 50  0001 C CNN "LCSC"
 	1    3500 1900
 	1    0    0    -1
@@
 F 0 "R10" H 3559 2246 50  0000 L CNN
 F 1 "2k2" H 3559 2155 50  0000 L CNN
-F 2 "Collins-FMS-3000:Perfect_0402" H 3500 2200 50  0001 C CNN
+F 2 "Resistor_SMD:R_0603_1608Metric" H 3500 2200 50  0001 C CNN
 F 3 "~" H 3500 2200 50  0001 C CNN
+F 4 "0603" H 3500 2200 50  0001 C CNN "JLC"
+F 5 "C22939" H 3500 2200 50  0001 C CNN "LCSC"
 	1    3500 2200
 	1    0    0    -1
@@
 F 0 "R11" H 3559 2546 50  0000 L CNN
 F 1 "2k2" H 3559 2455 50  0000 L CNN
-F 2 "Collins-FMS-3000:Perfect_0402" H 3500 2500 50  0001 C CNN
+F 2 "Resistor_SMD:R_0603_1608Metric" H 3500 2500 50  0001 C CNN
 F 3 "~" H 3500 2500 50  0001 C CNN
+F 4 "0603" H 3500 2500 50  0001 C CNN "JLC"
+F 5 "C22939" H 3500 2500 50  0001 C CNN "LCSC"
 	1    3500 2500
 	1    0    0    -1
@@
 F 0 "R12" H 3559 2846 50  0000 L CNN
 F 1 "2k2" H 3559 2755 50  0000 L CNN
-F 2 "Collins-FMS-3000:Perfect_0402" H 3500 2800 50  0001 C CNN
+F 2 "Resistor_SMD:R_0603_1608Metric" H 3500 2800 50  0001 C CNN
 F 3 "~" H 3500 2800 50  0001 C CNN
+F 4 "0603" H 3500 2800 50  0001 C CNN "JLC"
+F 5 "C22939" H 3500 2800 50  0001 C CNN "LCSC"
 	1    3500 2800
 	1    0    0    -1
@@
 F 0 "R13" H 3559 3146 50  0000 L CNN
 F 1 "2k2" H 3559 3055 50  0000 L CNN
-F 2 "Collins-FMS-3000:Perfect_0402" H 3500 3100 50  0001 C CNN
+F 2 "Resistor_SMD:R_0603_1608Metric" H 3500 3100 50  0001 C CNN
 F 3 "~" H 3500 3100 50  0001 C CNN
+F 4 "0603" H 3500 3100 50  0001 C CNN "JLC"
+F 5 "C22939" H 3500 3100 50  0001 C CNN "LCSC"
 	1    3500 3100
 	1    0    0    -1
@@
 F 0 "R14" H 3559 3446 50  0000 L CNN
 F 1 "2k2" H 3559 3355 50  0000 L CNN
-F 2 "Collins-FMS-3000:Perfect_0402" H 3500 3400 50  0001 C CNN
+F 2 "Resistor_SMD:R_0603_1608Metric" H 3500 3400 50  0001 C CNN
 F 3 "~" H 3500 3400 50  0001 C CNN
+F 4 "0603" H 3500 3400 50  0001 C CNN "JLC"
+F 5 "C22939" H 3500 3400 50  0001 C CNN "LCSC"
 	1    3500 3400
 	1    0    0    -1
@@
 F 0 "R15" H 3559 3746 50  0000 L CNN
 F 1 "2k2" H 3559 3655 50  0000 L CNN
-F 2 "Collins-FMS-3000:Perfect_0402" H 3500 3700 50  0001 C CNN
+F 2 "Resistor_SMD:R_0603_1608Metric" H 3500 3700 50  0001 C CNN
 F 3 "~" H 3500 3700 50  0001 C CNN
+F 4 "0603" H 3500 3700 50  0001 C CNN "JLC"
+F 5 "C22939" H 3500 3700 50  0001 C CNN "LCSC"
 	1    3500 3700
 	1    0    0    -1
@@
 F 0 "R16" H 3559 4046 50  0000 L CNN
 F 1 "2k2" H 3559 3955 50  0000 L CNN
-F 2 "Collins-FMS-3000:Perfect_0402" H 3500 4000 50  0001 C CNN
+F 2 "Resistor_SMD:R_0603_1608Metric" H 3500 4000 50  0001 C CNN
 F 3 "~" H 3500 4000 50  0001 C CNN
+F 4 "0603" H 3500 4000 50  0001 C CNN "JLC"
+F 5 "C22939" H 3500 4000 50  0001 C CNN "LCSC"
 	1    3500 4000
 	1    0    0    -1
@@
 F 0 "R17" H 3559 4346 50  0000 L CNN
 F 1 "2k2" H 3559 4255 50  0000 L CNN
-F 2 "Collins-FMS-3000:Perfect_0402" H 3500 4300 50  0001 C CNN
+F 2 "Resistor_SMD:R_0603_1608Metric" H 3500 4300 50  0001 C CNN
 F 3 "~" H 3500 4300 50  0001 C CNN
+F 4 "0603" H 3500 4300 50  0001 C CNN "JLC"
+F 5 "C22939" H 3500 4300 50  0001 C CNN "LCSC"
 	1    3500 4300
 	1    0    0    -1
@@
 F 0 "R18" H 3559 4646 50  0000 L CNN
 F 1 "2k2" H 3559 4555 50  0000 L CNN
-F 2 "Collins-FMS-3000:Perfect_0402" H 3500 4600 50  0001 C CNN
+F 2 "Resistor_SMD:R_0603_1608Metric" H 3500 4600 50  0001 C CNN
 F 3 "~" H 3500 4600 50  0001 C CNN
+F 4 "0603" H 3500 4600 50  0001 C CNN "JLC"
+F 5 "C22939" H 3500 4600 50  0001 C CNN "LCSC"
 	1    3500 4600
 	1    0    0    -1
@@
 F 0 "R19" H 3559 4946 50  0000 L CNN
 F 1 "2k2" H 3559 4855 50  0000 L CNN
-F 2 "Collins-FMS-3000:Perfect_0402" H 3500 4900 50  0001 C CNN
+F 2 "Resistor_SMD:R_0603_1608Metric" H 3500 4900 50  0001 C CNN
 F 3 "~" H 3500 4900 50  0001 C CNN
+F 4 "0603" H 3500 4900 50  0001 C CNN "JLC"
+F 5 "C22939" H 3500 4900 50  0001 C CNN "LCSC"
 	1    3500 4900
 	1    0    0    -1

Commit message: Fix pull-up resistor value Fixes #14
Parts:
- R10, R11, R12, R13, R14, R15, R16, R17, R18, R19, R8, R9: LCSC C22939 -> C4190
Changed lines of the file:
@@
 F 3 "~" H 3500 1600 50  0001 C CNN
 F 4 "0603" H 3500 1600 50  0001 C CNN "JLC"
-F 5 "C22939" H 3500 1600 50  0001 C CNN "LCSC"
+F 5 "C4190" H 3500 1600 50  0001 C CNN "LCSC"
 	1    3500 1600
 	1    0    0    -1
@@
 F 3 "~" H 3500 1900 50  0001 C CNN
 F 4 "0603" H 3500 1900 50  0001 C CNN "JLC"
-F 5 "C22939" H 3500 1900 50  0001 C CNN "LCSC"
+F 5 "C4190" H 3500 1900 50  0001 C CNN "LCSC"
 	1    3500 1900
 	1    0    0    -1
@@
 F 3 "~" H 3500 2200 50  0001 C CNN
 F 4 "0603" H 3500 2200 50  0001 C CNN "JLC"
-F 5 "C22939" H 3500 2200 50  0001 C CNN "LCSC"
+F 5 "C4190" H 3500 2200 50  0001 C CNN "LCSC"
 	1    3500 2200
 	1    0    0    -1
@@
 F 3 "~" H 3500 2500 50  0001 C CNN
 F 4 "0603" H 3500 2500 50  0001 C CNN "JLC"
-F 5 "C22939" H 3500 2500 50  0001 C CNN "LCSC"
+F 5 "C4190" H 3500 2500 50  0001 C CNN "LCSC"
 	1    3500 2500
 	1    0    0    -1
@@
 F 3 "~" H 3500 2800 50  0001 C CNN
 F 4 "0603" H 3500 2800 50  0001 C CNN "JLC"
-F 5 "C22939" H 3500 2800 50  0001 C CNN "LCSC"
+F 5 "C4190" H 3500 2800 50  0001 C CNN "LCSC"
 	1    3500 2800
 	1    0    0    -1
@@
 F 3 "~" H 3500 3100 50  0001 C CNN
 F 4 "0603" H 3500 3100 50  0001 C CNN "JLC"
-F 5 "C22939" H 3500 3100 50  0001 C CNN "LCSC"
+F 5 "C4190" H 3500 3100 50  0001 C CNN "LCSC"
 	1    3500 3100
 	1    0    0    -1
@@
 F 3 "~" H 3500 3400 50  0001 C CNN
 F 4 "0603" H 3500 3400 50  0001 C CNN "JLC"
-F 5 "C22939" H 3500 3400 50  0001 C CNN "LCSC"
+F 5 "C4190" H 3500 3400 50  0001 C CNN "LCSC"
 	1    3500 3400
 	1    0    0    -1
@@
 F 3 "~" H 3500 3700 50  0001 C CNN
 F 4 "0603" H 3500 3700 50  0001 C CNN "JLC"
-F 5 "C22939" H 3500 3700 50  0001 C CNN "LCSC"
+F 5 "C4190" H 3500 3700 50  0001 C CNN "LCSC"
 	1    3500 3700
 	1    0    0    -1
@@
 F 3 "~" H 3500 4000 50  0001 C CNN
 F 4 "0603" H 3500 4000 50  0001 C CNN "JLC"
-F 5 "C22939" H 3500 4000 50  0001 C CNN "LCSC"
+F 5 "C4190" H 3500 4000 50  0001 C CNN "LCSC"
 	1    3500 4000
 	1    0    0    -1
@@
 F 3 "~" H 3500 4300 50  0001 C CNN
 F 4 "0603" H 3500 4300 50  0001 C CNN "JLC"
-F 5 "C22939" H 3500 4300 50  0001 C CNN "LCSC"
+F 5 "C4190" H 3500 4300 50  0001 C CNN "LCSC"
 	1    3500 4300
 	1    0    0    -1
@@
 F 3 "~" H 3500 4600 50  0001 C CNN
 F 4 "0603" H 3500 4600 50  0001 C CNN "JLC"
-F 5 "C22939" H 3500 4600 50  0001 C CNN "LCSC"
+F 5 "C4190" H 3500 4600 50  0001 C CNN "LCSC"
 	1    3500 4600
 	1    0    0    -1
@@
 F 3 "~" H 3500 4900 50  0001 C CNN
 F 4 "0603" H 3500 4900 50  0001 C CNN "JLC"
-F 5 "C22939" H 3500 4900 50  0001 C CNN "LCSC"
+F 5 "C4190" H 3500 4900 50  0001 C CNN "LCSC"
 	1    3500 4900
 	1    0    0    -1
