File: ButtonMatrix.kicad_sch (KiCad schematic)
At the start: 69 parts, among them SW1 SW_Push_LED, SW10 SW_Push_LED, SW11 SW_Push_LED, SW12 SW_Push_LED, SW13 SW_Push_LED, SW14 SW_Push_LED, SW15 SW_Push_LED, SW16 SW_Push_LED, SW17 SW_Push_LED, SW18 SW_Push_LED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

Commit message: Lots of pre-work before replacing RP2040 layout
Parts:
- SW1, SW10, SW11, SW12, SW13, SW14, SW15, SW16, SW17, SW18, SW19, SW2, SW20, SW21, SW22, SW23, SW24, SW25, SW26, SW27, SW28, SW29, SW3, SW30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: footprint Collins-FMS-3000:SW_PUSH_6mm -> Custom_Footprints:SW_PUSH_LED_THT
