File: LEDMatrix.kicad_sch (KiCad schematic)
At the start: 69 parts, among them SW1 SW_Push_LED, SW10 SW_Push_LED, SW11 SW_Push_LED, SW12 SW_Push_LED, SW13 SW_Push_LED, SW14 SW_Push_LED, SW15 SW_Push_LED, SW16 SW_Push_LED, SW17 SW_Push_LED, SW18 SW_Push_LED, SW19 SW_Push_LED, SW2 SW_Push_LED, SW20 SW_Push_LED, SW21 SW_Push_LED, SW22 SW_Push_LED, SW23 SW_Push_LED, SW24 SW_Push_LED, SW25 SW_Push_LED, SW26 SW_Push_LED, SW27 SW_Push_LED, SW28 SW_Push_LED, SW29 SW_Push_LED, SW3 SW_Push_LED, SW30 SW_Push_LED, SW31 SW_Push_LED, SW32 SW_Push_LED, SW33 SW_Push_LED, SW34 SW_Push_LED, SW35 SW_Push_LED, SW36 SW_Push_LED, SW37 SW_Push_LED, SW38 SW_Push_LED, SW39 SW_Push_LED, SW4 SW_Push_LED, SW40 SW_Push_LED, SW41 SW_Push_LED, SW42 SW_Push_LED, SW43 SW_Push_LED, SW44 SW_Push_LED, SW45 SW_Push_LED, SW46 SW_Push_LED, SW47 SW_Push_LED, SW48 SW_Push_LED, SW49 SW_Push_LED, SW5 SW_Push_LED, SW50 SW_Push_LED, SW51 SW_Push_LED, SW52 SW_Push_LED, SW53 SW_Push_LED, SW54 SW_Push_LED, SW55 SW_Push_LED, SW56 SW_Push_LED, SW57 SW_Push_LED, SW58 SW_Push_LED, SW59 SW_Push_LED, SW6 SW_Push_LED, SW60 SW_Push_LED, SW61 SW_Push_LED, SW62 SW_Push_LED, SW63 SW_Push_LED, SW64 SW_Push_LED, SW65 SW_Push_LED, SW66 SW_Push_LED, SW67 SW_Push_LED, SW68 SW_Push_LED, SW69 SW_Push_LED, SW7 SW_Push_LED, SW8 SW_Push_LED, SW9 SW_Push_LED

Commit message: JLCPCB rotation cleanup, kibot script fixes
Other:
- title: (none) -> Collins FMS 3000
Changed lines of the file:
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@@
 (kicad_sch (version 20211123) (generator eeschema)
   (paper "A4")
+  (title_block
+    (title "Collins FMS 3000")
+    (date "2022-11-02")
+    (rev "")
+  )
   (junction (at 31.75 105.41) (diameter 0) (color 0 0 0 0)
   )

Commit message: Keyboard driver (#25)
* Lots of pre-work before replacing RP2040 layout

* New RP2040 layout added

* FULLY ROUTED

* Clean up schematic

* More trace cleanup

* Final trace cleanup

Co-authored-by: Neil Enns <{ID}+{username}@users.noreply.github.com>
Parts:
- added C22, C23, C24, C28: 470nf, Custom_Footprints:Perfect_0402, symbol Device:C_Small
- added C25, C26, C27: 100nf, Custom_Footprints:Perfect_0402, symbol Device:C_Small
- added R6: 47k, Custom_Footprints:Perfect_0402, symbol Device:R_Small
- added R7: 100k, Resistor_SMD:R_0603_1608Metric, symbol Device:R_Small
- added U4: IS31FL3733B, Package_QFP:TQFP-48-1EP_7x7mm_P0.5mm_EP5x5mm_ThermalVias, symbol Collins-FMS-3000:IS31FL3733B
- SW1, SW10, SW11, SW12, SW13, SW14, SW15, SW16, SW17, SW18, SW19, SW2, SW20, SW21, SW22, SW23, SW24, SW25, SW26, SW27, SW28, SW29, SW3, SW30, SW31, SW32, SW33, SW34, SW35, SW36, SW37, SW38, SW39, SW4, SW40, SW41, SW42, SW43, SW44, SW45, SW46, SW47, SW48, SW49, SW5, SW50, SW51, SW52, SW53, SW54, SW55, SW56, SW57, SW58, SW59, SW6, SW60, SW61, SW62, SW63, SW64, SW65, SW66, SW67, SW68, SW69, SW7, SW8, SW9: footprint Collins-FMS-3000:SW_PUSH_6mm -> Custom_Footprints:SW_PUSH_LED_THT
Connections:
- net CS1: now also U4.16 (CS1)
- net CS10: now also U4.26 (CS10)
- net CS11: now also U4.27 (CS11)
- net CS12: now also U4.28 (CS12)
- net CS2: now also U4.17 (CS2)
- net CS3: now also U4.18 (CS3)
- net CS4: now also U4.19 (CS4)
- net CS5: now also U4.21 (CS5)
- net CS6: now also U4.22 (CS6)
- net CS7: now also U4.23 (CS7)
- net CS8: now also U4.24 (CS8)
- net CS9: now also U4.25 (CS9)
- net SW1: now also U4.2 (SW1)
- net SW10: now also U4.13 (SW10)
- net SW11: now also U4.14 (SW11)
- net SW12: now also U4.15 (SW12)
- net SW2: now also U4.3 (SW2)
- net SW3: now also U4.4 (SW3)
- net SW4: now also U4.6 (SW4)
- net SW5: now also U4.7 (SW5)
- net SW6: now also U4.8 (SW6)
- net SW7: now also U4.9 (SW7)
- net SW8: now also U4.10 (SW8)
- net SW9: now also U4.11 (SW9)
- new net: R6.1, U4.35 (ISET)
- new net: R7.1, U4.47 (IICRST)
- new net +3V3: C22.1, C23.1, C24.1, C25.1, C26.1, C27.1, C28.1, U4.20 (PVCC), U4.29 (PVCC), U4.37 (AVCC), U4.38 (DVCC), U4.39 (VIO)
- new net GND: C22.2, C23.2, C24.2, C25.2, C26.2, C27.2, C28.2, R6.2, R7.2, U4.12 (PGND), U4.34 (AGND), U4.43 (ADDR_2), U4.44 (ADDR_1), U4.48 (GND), U4.49 (GND), U4.5 (PGND)
- new net I2C_SCL: U4.42 (SCL)
- new net I2C_SDA: U4.41 (SDA)
- new net LED_INTB: U4.45 (INTB)
- new net SDB: U4.46 (SDB)
- no-connect marks 0 -> 5
Other:
- note added: "I2C address: 0x50"
- moved on the sheet: SW10B, SW11B, SW12B, SW13B, SW14B, SW15B, SW16B, SW17B, SW18B, SW19B, SW1B, SW20B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

Commit message: Clean up the schematic
Other:
- note added: "Button LEDs"
- note added: "LED driver"
- moved on the sheet: C22, C23, C24, C25, C26, C27, C28, R6, R7, SW10B, SW11B, SW12B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

Commit message: Renumber buttons to match key array position
Parts:
- renumbered SW66 to SW1, SW55 to SW11, SW51 to SW12, SW46 to SW13, SW41 to SW14, SW36 to SW15, SW31 to SW16, SW26 to SW17, SW21 to SW18, SW16 to SW19, SW50 to SW2, SW11 to SW20, SW56 to SW21, SW52 to SW22, SW47 to SW23, SW42 to SW24, SW37 to SW25, SW32 to SW26, SW22 to SW28, SW17 to SW29, SW45 to SW3, SW12 to SW30, SW57 to SW31, SW53 to SW32, SW48 to SW33, SW43 to SW34, SW38 to SW35, SW33 to SW36, SW28 to SW37, SW23 to SW38, SW18 to SW39, SW40 to SW4, SW13 to SW40, SW58 to SW41, SW54 to SW42, SW49 to SW43, SW39 to SW45, SW34 to SW46, SW29 to SW47, SW24 to SW48, SW19 to SW49, SW35 to SW5, SW14 to SW50, SW64 to SW51, SW65 to SW52, SW69 to SW53, SW67 to SW54, SW68 to SW55, SW10 to SW56, SW9 to SW57, SW8 to SW58, SW7 to SW59, SW30 to SW6, SW6 to SW60, SW59 to SW61, SW60 to SW62, SW61 to SW63, SW62 to SW64, SW63 to SW65, SW5 to SW66, SW4 to SW67, SW3 to SW68, SW2 to SW69, SW25 to SW7, SW1 to SW70, SW20 to SW8, SW15 to SW9
