File: RP2040.kicad_sch (KiCad schematic)
At the start: 28 parts, among them J1 USB_B_Micro, J2 Conn_01x02, U1 AMS1117-3.3, U5 W25Q128JVS, U6 RP2040, Y1 X322512MSB4SI

Commit message: Clean up schematic
Parts:
- C13: value 1UF -> 1uF; MPN - JLCPCB C1525 -> C52923
- C8: value 100nF -> 1uF; MPN - JLCPCB C1525 -> C52923
Changed lines of the file:
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@@
       (effects (font (size 1.27 1.27)) (justify left))
     )
-    (property "Value" "100nF" (id 1) (at 83.566 67.818 0)
+    (property "Value" "1uF" (id 1) (at 83.566 67.818 0)
       (effects (font (size 1.27 1.27)) (justify left))
     )
@@
       (effects (font (size 1.27 1.27)) hide)
     )
-    (property "MPN - JLCPCB" "C1525" (id 6) (at 80.645 66.675 0)
+    (property "MPN - JLCPCB" "C52923" (id 6) (at 80.645 66.675 0)
       (effects (font (size 1.27 1.27)) hide)
     )
@@
       (effects (font (size 1.27 1.27)) (justify left))
     )
-    (property "Value" "1UF" (id 1) (at 208.661 27.813 0)
+    (property "Value" "1uF" (id 1) (at 208.661 27.813 0)
       (effects (font (size 1.27 1.27)) (justify left))
     )
@@
       (effects (font (size 1.27 1.27)) hide)
     )
-    (property "MPN - JLCPCB" "C1525" (id 6) (at 205.74 26.67 0)
-      (effects (font (size 1.27 1.27)) hide)
-    )
+    (property "MPN - JLCPCB" "C52923" (id 6) (at 205.74 26.67 0)
+      (effects (font (size 1.27 1.27)) hide)
+    )

Commit message: Add debug connector
Parts:
- added J4: TC2030-IDC-NL, Connector:Tag-Connect_TC2030-IDC-NL_2x03_P1.27mm_Vertical, symbol Custom_Symbols:TC2030-IDC-NL
- added R13: 10k, Custom_Footprints:Perfect_0402, symbol Device:R_Small
Connections:
- net +3V3: now also R13.1
- net GND: now also J4.6 (Pin_6)
- net SWCLK: now also J4.5 (Pin_5)
- net SWD: now also J4.3 (Pin_3)
- net RUN renamed ~{RST}
- net ~{RST}: now also J4.1 (Pin_1), R13.2
Other:
- note added: "Debug connector"
Changed lines of the file:
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@@
   (junction (at 228.6 33.02) (diameter 0) (color 0 0 0 0)
+  )
+  (junction (at 134.62 125.73) (diameter 0) (color 0 0 0 0)
   )
   (junction (at 186.69 41.91) (diameter 0) (color 0 0 0 0)
@@
     (stroke (width 0) (type default) (color 0 0 0 0))
   )
+  (polyline (pts (xy 100.33 132.715) (xy 100.33 108.585))
+    (stroke (width 0) (type default) (color 0 0 0 0))
+  )
   (wire (pts (xy 196.85 20.32) (xy 196.85 21.59))
     (stroke (width 0) (type default) (color 0 0 0 0))
@@
     (stroke (width 0) (type default) (color 0 0 0 0))
   )
+  (polyline (pts (xy 74.93 132.715) (xy 100.33 132.715))
+    (stroke (width 0) (type default) (color 0 0 0 0))
+  )
   (wire (pts (xy 240.03 21.59) (xy 251.46 21.59))
     (stroke (width 0) (type default) (color 0 0 0 0))
@@
     (stroke (width 0) (type default) (color 0 0 0 0))
   )
+  (polyline (pts (xy 83.185 108.585) (xy 74.93 108.585))
+    (stroke (width 0) (type default) (color 0 0 0 0))
+  )
   (polyline (pts (xy 90.805 49.53) (xy 90.805 17.145))
     (stroke (width 0) (type default) (color 0 0 0 0))
@@
     (stroke (width 0) (type default) (color 0 0 0 0))
   )
+  (polyline (pts (xy 74.93 108.585) (xy 74.93 132.715))
+    (stroke (width 0) (type default) (color 0 0 0 0))
+  )
   (polyline (pts (xy 13.97 17.145) (xy 13.97 49.53))
     (stroke (width 0) (type default) (color 0 0 0 0))
   )
+  (wire (pts (xy 76.2 125.73) (xy 83.82 125.73))
+    (stroke (width 0) (type default) (color 0 0 0 0))
+  )
   (wire (pts (xy 262.89 33.02) (xy 274.32 33.02))
     (stroke (width 0) (type default) (color 0 0 0 0))
@@
     (stroke (width 0) (type default) (color 0 0 0 0))
   )
+  (polyline (pts (xy 83.185 108.585) (xy 100.33 108.585))
+    (stroke (width 0) (type default) (color 0 0 0 0))
+  )
   (wire (pts (xy 39.37 114.935) (xy 39.37 113.665))
     (stroke (width 0) (type default) (color 0 0 0 0))
@@
     (stroke (width 0) (type default) (color 0 0 0 0))
   )
+  (wire (pts (xy 76.2 123.19) (xy 83.82 123.19))
+    (stroke (width 0) (type default) (color 0 0 0 0))
+  )
   (polyline (pts (xy 13.97 108.585) (xy 13.97 132.715))
     (stroke (width 0) (type default) (color 0 0 0 0))
@@
     (stroke (width 0) (type default) (color 0 0 0 0))
   )
+  (wire (pts (xy 128.27 125.73) (xy 134.62 125.73))
+    (stroke (width 0) (type default) (color 0 0 0 0))
+  )
   (polyline (pts (xy 13.97 103.505) (xy 105.41 103.505))
     (stroke (width 0) (type default) (color 0 0 0 0))
@@
     (stroke (width 0) (type default) (color 0 0 0 0))
   )
+  (wire (pts (xy 76.2 120.65) (xy 83.82 120.65))
+    (stroke (width 0) (type default) (color 0 0 0 0))
+  )
   (wire (pts (xy 212.09 90.17) (xy 227.33 90.17))
     (stroke (width 0) (type default) (color 0 0 0 0))
@@
   )
   (text "Crystal" (at 13.97 107.315 0)
+    (effects (font (size 1.27 1.27)) (justify left bottom))
+  )
+  (text "Debug connector" (at 74.93 107.95 0)
     (effects (font (size 1.27 1.27)) (justify left bottom))
   )
@@
     (effects (font (size 1.27 1.27)) (justify left bottom))
   )
+  (label "~{RST}" (at 76.2 120.65 0)
+    (effects (font (size 1.27 1.27)) (justify left bottom))
+  )
   (label "USB_D_R-" (at 212.725 64.77 0)
     (effects (font (size 1.27 1.27)) (justify left bottom))
@@
     (effects (font (size 1.27 1.27)) (justify left bottom))
   )
-  (label "RUN" (at 134.62 125.73 0)
+  (label "~{RST}" (at 128.27 125.73 0)
     (effects (font (size 1.27 1.27)) (justify left bottom))
   )
@@
   (label "USB_D+" (at 245.11 57.15 180)
     (effects (font (size 1.27 1.27)) (justify right bottom))
+  )
+  (label "SWD" (at 76.2 123.19 0)
+    (effects (font (size 1.27 1.27)) (justify left bottom))
+  )
+  (label "SWCLK" (at 76.2 125.73 0)
+    (effects (font (size 1.27 1.27)) (justify left bottom))
   )
   (label "QSPI_SS" (at 50.165 85.725 0)
@@
     (pin "2")
   )
+  (symbol (lib_id "power:+3V3") (at 134.62 120.65 0) (unit 1)
+    (in_bom yes) (on_board yes) (fields_autoplaced)
+    (property "Reference" "#PWR011" (id 0) (at 134.62 124.46 0)
+      (effects (font (size 1.27 1.27)) hide)
+    )
+    (property "Value" "+3V3" (id 1) (at 134.62 115.57 0))
+    (property "Footprint" "" (id 2) (at 134.62 120.65 0)
+      (effects (font (size 1.27 1.27)) hide)
+    )
+    (property "Datasheet" "" (id 3) (at 134.62 120.65 0)
+      (effects (font (size 1.27 1.27)) hide)
+    )
+    (pin "1")
+  )
   (symbol (lib_id "Device:C") (at 80.645 66.675 0) (unit 1)
     (in_bom yes) (on_board yes)
@@
     (pin "2")
   )
+  (symbol (lib_id "Custom_Symbols:TC2030-IDC-NL") (at 90.17 123.19 0) (unit 1)
+    (in_bom yes) (on_board yes) (fields_autoplaced)
+    (property "Reference" "J4" (id 0) (at 90.17 110.49 0))
+    (property "Value" "TC2030-IDC-NL" (id 1) (at 90.17 113.03 0))
+    (property "Footprint" "Connector:Tag-Connect_TC2030-IDC-NL_2x03_P1.27mm_Vertical" (id 2) (at 88.9 123.19 0)
+      (effects (font (size 1.27 1.27)) hide)
+    )
+    (property "Datasheet" "https://www.tag-connect.com/wp-content/uploads/bsk-pdf-manager/2019/12/TC2030-IDC-NL-Datasheet-Rev-B.pdf" (id 3) (at 90.17 137.16 0)
+      (effects (font (size 1.27 1.27)) hide)
+    )
+    (pin "1")
+    (pin "2")
+    (pin "3")
+    (pin "4")
+    (pin "5")
+    (pin "6")
+  )
   (symbol (lib_id "Device:R") (at 43.815 85.725 270) (unit 1)
     (in_bom yes) (on_board yes)
@@
     (pin "2")
   )
+  (symbol (lib_id "Device:R_Small") (at 134.62 123.19 0) (unit 1)
+    (in_bom yes) (on_board yes) (fields_autoplaced)
+    (property "Reference" "R13" (id 0) (at 137.16 121.9199 0)
+      (effects (font (size 1.27 1.27)) (justify left))
+    )
+    (property "Value" "10k" (id 1) (at 137.16 124.4599 0)
+      (effects (font (size 1.27 1.27)) (justify left))
+    )
+    (property "Footprint" "Custom_Footprints:Perfect_0402" (id 2) (at 134.62 123.19 0)
+      (effects (font (size 1.27 1.27)) hide)
+    )
+    (property "Datasheet" "~" (id 3) (at 134.62 123.19 0)
+      (effects (font (size 1.27 1.27)) hide)
+    )
+    (property "MPN - JLCPCB" "C25744" (id 4) (at 134.62 123.19 0)
+      (effects (font (size 1.27 1.27)) hide)
+    )
+    (pin "1")
+    (pin "2")
+  )
   (symbol (lib_id "power:+1V1") (at 160.02 20.32 0) (unit 1)
     (in_bom yes) (on_board yes)
@@
     (pin "2")
   )
+  (symbol (lib_id "power:GND") (at 96.52 125.73 0) (unit 1)
+    (in_bom yes) (on_board yes) (fields_autoplaced)
+    (property "Reference" "#PWR07" (id 0) (at 96.52 132.08 0)
+      (effects (font (size 1.27 1.27)) hide)
+    )
+    (property "Value" "GND" (id 1) (at 96.52 130.175 0))
+    (property "Footprint" "" (id 2) (at 96.52 125.73 0)
+      (effects (font (size 1.27 1.27)) hide)
+    )
+    (property "Datasheet" "" (id 3) (at 96.52 125.73 0)
+      (effects (font (size 1.27 1.27)) hide)
+    )
+    (pin "1")
+  )
   (symbol (lib_id "power:+3V3") (at 250.19 70.485 0) (unit 1)
